File: Power.kicad_sch (KiCad schematic)
At the start: 88 parts, among them P10 CONN_1, P11 CONN_10X2, P12 POWER_SW, P2 CONN_1, P21 CONN_1, P22 CONN_1, P23 CONN_1, P3 CONN_1, P4 CONN_1, P5 CONN_1, P6 CONN_1, P7 CONN_1, P8 CONN_1, P9 CONN_1, SW1 POWER, U12 74LS74, U14 74LS125, U18 74LS32, U19 74HCT14, U2 74LS14, U26 74LS06, U32 74LS139, U33 74LS10, U34 74LS393, U39 74LS04, U49 74LS07N, U5 74LS02, U59 74LS32, U6 74LS32, U63 74LS14, U7 74LS32, U8 74LS08

Commit message: rev 1.0
Parts:
- removed U59: 74LS32, Custom:STD_DDW_DIP14, symbol 74xx:74LS32
- added RR1: 4700, Custom:STD_DDW_SIP10, symbol Device:R_Network09_US
- RR5: footprint Resistor_THT:R_Array_SIP10 -> Custom:STD_DDW_SIP10
Connections:
- net +5V: now also RR1.1 (common)
- new net /BUSRQ: RR1.4 (R3)
- new net /CPU_INT0: RR1.2 (R1)
- new net /CPU_INT1: RR1.3 (R2)
- new net /TRG1-A: RR1.5 (R4)
- new net /TRG1-B: RR1.6 (R5)
- new net /TRG2-A: RR1.7 (R6)
- new net /TRG2-B: RR1.8 (R7)
- no-connect marks 10 -> 12
