File: floppy.kicad_sch (KiCad schematic)
At the start: 11 parts, among them P27 FLOPPY, P41 OSC_FDC, U32 74LS139, U33 74LS10, U39 74LS04, U59 74LS32, U61 WD37C65BJM, U8 74LS08

Commit message: rev 1.0
Parts:
- RP1: footprint Resistor_THT:R_Array_SIP9 -> Custom:STD_DDW_SIP9
- renumbered U59 to U6
Connections:
- net A1: now also U6.5; no longer U6.13
- net /CS_FDC: now also U6.1, U6.4; no longer U6.12, U6.9
- net /TC: now also U6.3; no longer U6.8
- net at U61.3 (/CS): now also U6.6; no longer U6.11
- net at U39.2: now also U6.2; no longer U6.10
- net at U61.18 (/LDOR): now also U32.6 (O2); no longer U32.5 (O1)
- net at U61.19 (/LDCR): now also U32.5 (O1); no longer U32.6 (O2)
Changed lines of the file:
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@@
 	(title_block
 		(title "N8PC")
-		(date "2025-11-02")
-		(rev "000.8")
+		(date "2025-11-26")
+		(rev "000.9")
 		(comment 1 "https://github.com/danwerner21/N8PC")
 		(comment 2 "Based on work by Andrew Lynch and John Coffman")
@@
 	(wire
 		(pts
+			(xy 130.81 151.13) (xy 167.64 151.13)
+		)
+		(stroke
+			(width 0)
+			(type default)
+		)
+	)
+	(wire
+		(pts
 			(xy 289.56 129.54) (xy 289.56 156.21)
 		)
@@
 	(wire
 		(pts
-			(xy 130.81 151.13) (xy 166.37 151.13)
-		)
-		(stroke
-			(width 0)
-			(type default)
-		)
-	)
-	(wire
-		(pts
-			(xy 167.64 119.38) (xy 167.64 153.67)
-		)
-		(stroke
-			(width 0)
-			(type default)
-		)
-	)
-	(wire
-		(pts
 			(xy 182.88 146.05) (xy 177.8 146.05)
 		)
@@
 	(wire
 		(pts
+			(xy 167.64 119.38) (xy 167.64 151.13)
+		)
+		(stroke
+			(width 0)
+			(type default)
+		)
+	)
+	(wire
+		(pts
 			(xy 182.88 133.35) (xy 177.8 133.35)
 		)
@@
 	(wire
 		(pts
-			(xy 166.37 151.13) (xy 166.37 116.84)
-		)
-		(stroke
-			(width 0)
-			(type default)
-		)
-	)
-	(wire
-		(pts
 			(xy 281.94 121.92) (xy 279.4 124.46)
 		)
@@
 	(wire
 		(pts
+			(xy 130.81 153.67) (xy 166.37 153.67)
+		)
+		(stroke
+			(width 0)
+			(type default)
+		)
+	)
+	(wire
+		(pts
 			(xy 279.4 121.92) (xy 281.94 124.46)
 		)
@@
 	(wire
 		(pts
+			(xy 166.37 116.84) (xy 166.37 153.67)
+		)
+		(stroke
+			(width 0)
+			(type default)
+		)
+	)
+	(wire
+		(pts
 			(xy 222.25 161.29) (xy 294.64 161.29)
 		)
@@
 		(pts
 			(xy 294.64 161.29) (xy 304.8 161.29)
-		)
-		(stroke
-			(width 0)
-			(type default)
-		)
-	)
-	(wire
-		(pts
-			(xy 130.81 153.67) (xy 167.64 153.67)
 		)
 		(stroke
@@
 		(lib_id "74xx:74LS32")
 		(at 137.16 111.76 0)
-		(unit 4)
+		(unit 2)
 		(exclude_from_sim no)
 		(in_bom yes)
 		(on_board yes)
 		(dnp no)
-		(property "Reference" "U59"
+		(property "Reference" "U6"
 			(at 137.922 111.76 0)
 			(effects
@@
 			(project "N8PC"
 				(path "/d94f9d60-5ece-4752-b49c-b0d1c95f35bc/2083a38b-f429-4889-aed4-507d154b3f47"
-					(reference "U59")
-					(unit 4)
+					(reference "U6")
+					(unit 2)
 				)
 			)
@@
 		(lib_id "74xx:74LS32")
 		(at 137.16 124.46 0)
-		(unit 3)
+		(unit 1)
 		(exclude_from_sim no)
 		(in_bom yes)
 		(on_board yes)
 		(dnp no)
-		(property "Reference" "U59"
+		(property "Reference" "U6"
 			(at 137.668 124.46 0)
 			(effects
@@
 			(project "N8PC"
 				(path "/d94f9d60-5ece-4752-b49c-b0d1c95f35bc/2083a38b-f429-4889-aed4-507d154b3f47"
-					(reference "U59")
-					(unit 3)
+					(reference "U6")
+					(unit 1)
 				)
 			)
@@
 			)
 		)
-		(property "Footprint" "Resistor_THT:R_Array_SIP9"
+		(property "Footprint" "Custom:STD_DDW_SIP9"
 			(at 309.88 170.815 90)
 			(effects
