File: ide.kicad_sch (KiCad schematic)
At the start: 6 parts, among them K2 IDE_PWR, P29 PPIDE, P31 PARALLEL EXP, U38 8255, U63 74LS14

Commit message: rev 1.0
Parts:
- U38: footprint Package_DIP:DIP-40_W15.24mm -> Custom:STD_DDW_DIP40
Changed lines of the file:
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@@
 	(title_block
 		(title "N8PC")
-		(date "2025-11-02")
-		(rev "000.8")
+		(date "2025-11-26")
+		(rev "000.9")
 		(comment 1 "https://github.com/danwerner21/N8PC")
 		(comment 2 "Based on work by Andrew Lynch and John Coffman")
@@
 			)
 		)
-		(property "Footprint" "Package_DIP:DIP-40_W15.24mm"
+		(property "Footprint" "Custom:STD_DDW_DIP40"
 			(at 114.3 95.25 0)
 			(effects
