File: ramrom.kicad_sch (KiCad schematic)
At the start: 7 parts, among them K16 CONN_3, K18 CONN_3, K3 CONN_3, K4 CONN_3, K5 CONN_3, U13 27C080, U53 SRAM_512KO

Commit message: rev 1.0
Parts:
- U53: footprint Package_DIP:DIP-32_W15.24mm -> Custom:STD_DDW_DIP32
Changed lines of the file:
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@@
 	(title_block
 		(title "N8PC")
-		(date "2025-11-02")
-		(rev "000.8")
+		(date "2025-11-26")
+		(rev "000.9")
 		(comment 1 "https://github.com/danwerner21/N8PC")
 		(comment 2 "Based on work by Andrew Lynch and John Coffman")
@@
 			)
 		)
-		(property "Footprint" "Package_DIP:DIP-32_W15.24mm"
+		(property "Footprint" "Custom:STD_DDW_DIP32"
 			(at 187.96 64.77 0)
 			(effects
