File: serial.kicad_sch (KiCad schematic)
At the start: 21 parts, among them J17 TTL SERIAL CONSOLE, J18 TTL CONSOLE PWR, J19 TTL SERIAL CONSOLE, J20 TTL CONSOLE PWR, P13 SERIAL, P18 SERIAL, U10 MAX232, U35 MAX232

Commit message: rev 1.0
Connections:
- net SIN_TTL0: now also J17.4 (Pin_4); no longer J17.5 (Pin_5)
- net SIN_TTL1: now also J19.4 (Pin_4); no longer J19.5 (Pin_5)
- net SOUT_TTL0: now also J17.5 (Pin_5); no longer J17.4 (Pin_4)
- net SOUT_TTL1: now also J19.5 (Pin_5); no longer J19.4 (Pin_4)
Changed lines of the file:
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@@
 	(title_block
 		(title "N8PC")
-		(date "2025-11-02")
-		(rev "000.8")
+		(date "2025-11-26")
+		(rev "000.9")
 		(comment 1 "https://github.com/danwerner21/N8PC")
 		(comment 2 "Based on work by Andrew Lynch and John Coffman")
@@
 	(global_label "SIN_TTL1"
 		(shape output)
-		(at 257.81 106.68 0)
-		(fields_autoplaced yes)
-		(effects
-			(font
-				(size 1.27 1.27)
-			)
-			(justify left)
-		)
-		(property "Intersheetrefs" "${INTERSHEET_REFS}"
-			(at 268.4262 106.68 0)
+		(at 257.81 104.14 0)
+		(fields_autoplaced yes)
+		(effects
+			(font
+				(size 1.27 1.27)
+			)
+			(justify left)
+		)
+		(property "Intersheetrefs" "${INTERSHEET_REFS}"
+			(at 268.4262 104.14 0)
 			(effects
 				(font
@@
 	(global_label "SIN_TTL0"
 		(shape output)
-		(at 257.81 76.2 0)
-		(fields_autoplaced yes)
-		(effects
-			(font
-				(size 1.27 1.27)
-			)
-			(justify left)
-		)
-		(property "Intersheetrefs" "${INTERSHEET_REFS}"
-			(at 268.4262 76.2 0)
+		(at 257.81 73.66 0)
+		(fields_autoplaced yes)
+		(effects
+			(font
+				(size 1.27 1.27)
+			)
+			(justify left)
+		)
+		(property "Intersheetrefs" "${INTERSHEET_REFS}"
+			(at 268.4262 73.66 0)
 			(effects
 				(font
@@
 	(global_label "SOUT_TTL1"
 		(shape input)
-		(at 257.81 104.14 0)
-		(fields_autoplaced yes)
-		(effects
-			(font
-				(size 1.27 1.27)
-			)
-			(justify left)
-		)
-		(property "Intersheetrefs" "${INTERSHEET_REFS}"
-			(at 270.1195 104.14 0)
+		(at 257.81 106.68 0)
+		(fields_autoplaced yes)
+		(effects
+			(font
+				(size 1.27 1.27)
+			)
+			(justify left)
+		)
+		(property "Intersheetrefs" "${INTERSHEET_REFS}"
+			(at 270.1195 106.68 0)
 			(effects
 				(font
@@
 	(global_label "SOUT_TTL0"
 		(shape input)
-		(at 257.81 73.66 0)
-		(fields_autoplaced yes)
-		(effects
-			(font
-				(size 1.27 1.27)
-			)
-			(justify left)
-		)
-		(property "Intersheetrefs" "${INTERSHEET_REFS}"
-			(at 270.1195 73.66 0)
-			(effects
-				(font
+		(at 257.81 76.2 0)
+		(fields_autoplaced yes)
+		(effects
+			(font
+				(size 1.27 1.27)
+			)
+			(justify left)
+		)
+		(property "Intersheetrefs" "${INTERSHEET_REFS}"
+			(at 270.1195 76.2 0)
+			(effects
+				(font
